File: 01POWER.kicad_sch (KiCad schematic)
At the start: 1 part, among them U1 HPM6880IBD1

Commit message: 添加库 添加网络类
Connections:
- net GND: now reaches U1.A15 (VSS)
- net GND: now also U1.A21 (VSS), U1.A27 (VSS), U1.A3 (VSS), U1.A9 (VSS), U1.AA1 (VSS), U1.AA11 (VSS), U1.AA13 (VSS), U1.AA17 (VSS), U1.AA27 (VSS), U1.AA29 (VSS), U1.AA3 (VSS), U1.AD28 (VSS)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
