File: HPM6800_Core.kicad_sch (KiCad schematic)
At the start: 0 parts

Commit message: 添加库 添加网络类
Parts:
- added U1: HPM6880IBD1, HPM_footprints:BGA_417, symbol HPM6800:HPM6880IBD1
Connections:
- new net USB0_DN: U1.C3 (USB0_DN)
- new net USB0_DP: U1.B2 (USB0_DP)
